Commit message: add workflow trail test

File: figuer/urdf/figuer.xacro (robot description, xacro)
@@ -1,4 +1,5 @@
 <?xml version="1.0" encoding="utf-8"?>
-<robot  name="EG2-4C2" xmlns:xacro="http://www.ros.org/wiki/xacro">
+<robot  name="figuer" xmlns:xacro="http://www.ros.org/wiki/xacro">
+   <xacro:macro name="figuer" params="figure_name parent_link *origin rate">
   <link
     name="4C2_baselink">
@@ -23,22 +24,27 @@
       <geometry>
         <mesh
-          filename="package://EG2-4C2/meshes/4C2_baselink.STL" />
-      </geometry>
-      <material
-        name="">
-        <color
-          rgba="0.75294 0.75294 0.75294 1" />
-      </material>
-    </visual>
-    <collision>
-      <origin
-        xyz="0 0 0"
-        rpy="0 0 0" />
-      <geometry>
-        <mesh
-          filename="package://EG2-4C2/meshes/4C2_baselink.STL" />
-      </geometry>
-    </collision>
-  </link>
+          filename="package://figuer/meshes/4C2_baselink.STL" />
+      </geometry>
+      <material
+        name="">
+        <color
+          rgba="0.75294 0.75294 0.75294 1" />
+      </material>
+    </visual>
+    <collision>
+      <origin
+        xyz="0 0 0"
+        rpy="0 0 0" />
+      <geometry>
+        <mesh
+          filename="package://figuer/meshes/4C2_baselink.STL" />
+      </geometry>
+    </collision>
+  </link>
+  <joint name="${figure_name}_joint" type="fixed">
+      <parent link="${parent_link}"/>
+      <child link="4C2_baselink" />
+      <origin xyz="0 0 0" rpy="0 0 0"/>
+  </joint>
   <link
     name="4C2_Link1">
@@ -63,19 +69,19 @@
       <geometry>
         <mesh
-          filename="package://EG2-4C2/meshes/4C2_Link1.STL" />
-      </geometry>
-      <material
-        name="">
-        <color
-          rgba="0.75294 0.75294 0.75294 1" />
-      </material>
-    </visual>
-    <collision>
-      <origin
-        xyz="0 0 0"
-        rpy="0 0 0" />
-      <geometry>
-        <mesh
-          filename="package://EG2-4C2/meshes/4C2_Link1.STL" />
+          filename="package://figuer/meshes/4C2_Link1.STL" />
+      </geometry>
+      <material
+        name="">
+        <color
+          rgba="0.75294 0.75294 0.75294 1" />
+      </material>
+    </visual>
+    <collision>
+      <origin
+        xyz="0 0 0"
+        rpy="0 0 0" />
+      <geometry>
+        <mesh
+          filename="package://figuer/meshes/4C2_Link1.STL" />
       </geometry>
     </collision>
@@ -121,19 +127,19 @@
       <geometry>
         <mesh
-          filename="package://EG2-4C2/meshes/4C2_Link5.STL" />
-      </geometry>
-      <material
-        name="">
-        <color
-          rgba="0.75294 0.75294 0.75294 1" />
-      </material>
-    </visual>
-    <collision>
-      <origin
-        xyz="0 0 0"
-        rpy="0 0 0" />
-      <geometry>
-        <mesh
-          filename="package://EG2-4C2/meshes/4C2_Link5.STL" />
+          filename="package://figuer/meshes/4C2_Link5.STL" />
+      </geometry>
+      <material
+        name="">
+        <color
+          rgba="0.75294 0.75294 0.75294 1" />
+      </material>
+    </visual>
+    <collision>
+      <origin
+        xyz="0 0 0"
+        rpy="0 0 0" />
+      <geometry>
+        <mesh
+          filename="package://figuer/meshes/4C2_Link5.STL" />
       </geometry>
     </collision>
@@ -180,19 +186,19 @@
       <geometry>
         <mesh
-          filename="package://EG2-4C2/meshes/4C2_Link2.STL" />
-      </geometry>
-      <material
-        name="">
-        <color
-          rgba="0.75294 0.75294 0.75294 1" />
-      </material>
-    </visual>
-    <collision>
-      <origin
-        xyz="0 0 0"
-        rpy="0 0 0" />
-      <geometry>
-        <mesh
-          filename="package://EG2-4C2/meshes/4C2_Link2.STL" />
+          filename="package://figuer/meshes/4C2_Link2.STL" />
+      </geometry>
+      <material
+        name="">
+        <color
+          rgba="0.75294 0.75294 0.75294 1" />
+      </material>
+    </visual>
+    <collision>
+      <origin
+        xyz="0 0 0"
+        rpy="0 0 0" />
+      <geometry>
+        <mesh
+          filename="package://figuer/meshes/4C2_Link2.STL" />
       </geometry>
     </collision>
@@ -239,19 +245,19 @@
       <geometry>
         <mesh
-          filename="package://EG2-4C2/meshes/4C2_Link3.STL" />
-      </geometry>
-      <material
-        name="">
-        <color
-          rgba="0.75294 0.75294 0.75294 1" />
-      </material>
-    </visual>
-    <collision>
-      <origin
-        xyz="0 0 0"
-        rpy="0 0 0" />
-      <geometry>
-        <mesh
-          filename="package://EG2-4C2/meshes/4C2_Link3.STL" />
+          filename="package://figuer/meshes/4C2_Link3.STL" />
+      </geometry>
+      <material
+        name="">
+        <color
+          rgba="0.75294 0.75294 0.75294 1" />
+      </material>
+    </visual>
+    <collision>
+      <origin
+        xyz="0 0 0"
+        rpy="0 0 0" />
+      <geometry>
+        <mesh
+          filename="package://figuer/meshes/4C2_Link3.STL" />
       </geometry>
     </collision>
@@ -298,19 +304,19 @@
       <geometry>
         <mesh
-          filename="package://EG2-4C2/meshes/4C2_Link4.STL" />
-      </geometry>
-      <material
-        name="">
-        <color
-          rgba="0.75294 0.75294 0.75294 1" />
-      </material>
-    </visual>
-    <collision>
-      <origin
-        xyz="0 0 0"
-        rpy="0 0 0" />
-      <geometry>
-        <mesh
-          filename="package://EG2-4C2/meshes/4C2_Link4.STL" />
+          filename="package://figuer/meshes/4C2_Link4.STL" />
+      </geometry>
+      <material
+        name="">
+        <color
+          rgba="0.75294 0.75294 0.75294 1" />
+      </material>
+    </visual>
+    <collision>
+      <origin
+        xyz="0 0 0"
+        rpy="0 0 0" />
+      <geometry>
+        <mesh
+          filename="package://figuer/meshes/4C2_Link4.STL" />
       </geometry>
     </collision>
@@ -357,19 +363,19 @@
       <geometry>
         <mesh
-          filename="package://EG2-4C2/meshes/4C2_Link6.STL" />
-      </geometry>
-      <material
-        name="">
-        <color
-          rgba="0.75294 0.75294 0.75294 1" />
-      </material>
-    </visual>
-    <collision>
-      <origin
-        xyz="0 0 0"
-        rpy="0 0 0" />
-      <geometry>
-        <mesh
-          filename="package://EG2-4C2/meshes/4C2_Link6.STL" />
+          filename="package://figuer/meshes/4C2_Link6.STL" />
+      </geometry>
+      <material
+        name="">
+        <color
+          rgba="0.75294 0.75294 0.75294 1" />
+      </material>
+    </visual>
+    <collision>
+      <origin
+        xyz="0 0 0"
+        rpy="0 0 0" />
+      <geometry>
+        <mesh
+          filename="package://figuer/meshes/4C2_Link6.STL" />
       </geometry>
     </collision>
@@ -404,3 +410,4 @@
     </actuator>
   </transmission>
+</xacro:macro>
 </robot>

File: rm_description/urdf/RM65/rm_65.urdf.xacro (robot description, xacro)
@@ -3,5 +3,6 @@
 <xacro:include filename="$(find rm_description)/urdf/RM65/rm_65.transmission.xacro"/>
 <xacro:include filename="$(find rm_description)/urdf/RM65/rm_65.gazebo.xacro"/>
-<!-- <xacro:include filename="$(find rm_description)/urdf/EG2-4C2/urdf/EG2-4C2.urdf.xacro"/> -->
+<xacro:include filename="$(find realsense_ros_gazebo)/xacro/depthcam.xacro"/>
+<xacro:include filename="$(find rm_description)/urdf/RM65/gripper.xacro"/>
   <!-- Inertial matrix -->
   <xacro:macro name="inertial_matrix" params="mass">
@@ -447,4 +448,18 @@
 	<dynamics damping="50" friction="1"/>
   </joint>
+ <!-- gripper -->
+<!-- <xacro:simple_gripper gripper_name="gripper1" parent_link="Link6"
+                      finger_length="0.01" finger_width="0.01" finger_thickness="0.05">
+  <origin xyz="0 0 0.02" rpy="0 0 1.57"/>
+</xacro:simple_gripper>
+ -->
+<!-- <xacro:simple_gripper gripper_name="gripper1" parent_link="Link6"
+                      finger_length="0.1" finger_width="0.02" finger_thickness="0.01">
+  <origin xyz="0 0 1" rpy="0 0 0"/>
+</xacro:simple_gripper> -->
+<!-- realsense -->
+<xacro:realsense_d435 sensor_name="d435" parent_link="Link6" rate="10">
+   <origin rpy="3.1415 4.712 0 " xyz="0.07 0 0"/>
+</xacro:realsense_d435>
   <!-- Transmissions for ROS Control -->
   <xacro:macro name="transmission_block" params="joint_name">
